Commit message: new virtual system macro

File: kmr_iiwa_gazebo/urdf/kmr_iiwa.urdf.xacro (robot description, xacro)
@@ -7,5 +7,6 @@
   <xacro:include filename="$(find gz_virtual_base_system)/urdf/virtual_base_macro.urdf.xacro" />
   <!-- arguments -->
-  <xacro:arg name="robot_name" default="kmp_iiwa" />
+  <xacro:arg name="root_link" default="world"/> <!-- Put world for the gazebo model, odom for nav2 -->
+  <xacro:arg name="robot_name" default="kmr_iiwa" />
   <xacro:arg name="base_name" default="kmp" />
   <xacro:arg name="arm_name" default="iiwa" />
@@ -64,14 +65,5 @@
   </ros2_control> -->
   <!-- OPTION 3. virtual joints, virtual base system -->
-  <link name="odom">
-    <inertial>
-      <mass value="0.001"/>
-      <inertia
-        ixx="1e-6" ixy="0" ixz="0"
-        iyy="1e-6" iyz="0"
-        izz="1e-6"/>
-    </inertial>
-  </link>
-  <xacro:virtual_base_system world_link="odom" base_link="$(arg base_name)_base_link" />
+  <xacro:virtual_base_system root_link="$(arg root_link)" base_link="$(arg base_name)_base_link"/>
   <!-- Sensors -->
   <gazebo reference="$(arg base_name)_lidar_front_right_link">

Commit message: new urdf launch and conf for running without gazebo (e.g. real robot)

File: kmr_iiwa_gazebo/urdf/kmr_iiwa.urdf.xacro (robot description, xacro)
@@ -67,9 +67,9 @@
   <xacro:virtual_base_system root_link="$(arg root_link)" base_link="$(arg base_name)_base_link"/>
   <!-- Sensors -->
-  <gazebo reference="$(arg base_name)_lidar_front_right_link">
-  <sensor name="lidar_front_right" type="gpu_lidar">
-      <pose relative_to='$(arg base_name)_lidar_front_right_link'>0 0 0 0 0 0</pose>
-      <topic>$(arg robot_name)/lidar_front_right</topic>
-      <gz_frame_id>$(arg base_name)_lidar_front_right_link</gz_frame_id>
+  <gazebo reference="$(arg base_name)_scan_front_right_link">
+  <sensor name="scan_front_right" type="gpu_lidar">
+      <pose relative_to='$(arg base_name)_scan_front_right_link'>0 0 0 0 0 0</pose>
+      <topic>$(arg robot_name)/scan_front_right</topic>
+      <gz_frame_id>$(arg base_name)_scan_front_right_link</gz_frame_id>
       <!-- Response time 80 ms -->
       <update_rate>12.5</update_rate>
@@ -81,5 +81,7 @@
               <samples>540</samples>
               <resolution>1</resolution>
-              <!-- avoid the base -->
+              <!-- <min_angle>-2.35619442</min_angle>
+              <max_angle>2.3561944</max_angle> -->
+              <!-- Reduced to avoid taking the mobile base -->
               <min_angle>-2</min_angle>
               <max_angle>2</max_angle>
@@ -94,5 +96,5 @@
         <range>
             <min>0.05</min>
-            <max>30.0</max>
+            <max>29.0</max>
             <!-- Resolution (can be configured) 30 mm, 40 mm, 50 mm, 70 mm, 150 mm -->
             <resolution>0.05</resolution>
@@ -101,18 +103,22 @@
   </sensor>
   </gazebo>
-  <gazebo reference="$(arg base_name)_lidar_back_left_link">
-  <sensor name="lidar_back_left" type="gpu_lidar">
-      <pose relative_to='$(arg base_name)_lidar_back_left_link'>0 0 0 0 0 0</pose>
-      <topic>$(arg robot_name)/lidar_back_left</topic>
-      <gz_frame_id>$(arg base_name)_lidar_back_left_link</gz_frame_id>
+  <gazebo reference="$(arg base_name)_scan_back_left_link">
+  <sensor name="scan_back_left" type="gpu_lidar">
+      <pose relative_to='$(arg base_name)_scan_back_left_link'>0 0 0 0 0 0</pose>
+      <topic>$(arg robot_name)/scan_back_left</topic>
+      <gz_frame_id>$(arg base_name)_scan_back_left_link</gz_frame_id>
       <!-- Response time 80 ms -->
       <update_rate>12.5</update_rate>
-      <always_on>1</always_on>
+      <always_on>true</always_on>
       <visualize>true</visualize>
       <ray>
         <scan>
           <horizontal>
+              <!-- 270 deg / 0.5 deg -->
               <samples>540</samples>
               <resolution>1</resolution>
+              <!-- <min_angle>-2.35619442</min_angle>
+              <max_angle>2.3561944</max_angle> -->
+              <!-- Reduced to avoid taking the mobile base -->
               <min_angle>-2</min_angle>
               <max_angle>2</max_angle>
@@ -126,6 +132,6 @@
         </scan>
         <range>
-            <min>0.05</min>
-            <max>30.0</max>
+            <min>0.1</min>
+            <max>29.0</max>
             <!-- Resolution (can be configured) 30 mm, 40 mm, 50 mm, 70 mm, 150 mm -->
             <resolution>0.05</resolution>

File: kmr_iiwa_urdf/urdf/kmp200_macro.urdf.xacro (robot description, xacro)
@@ -32,16 +32,16 @@
   </link>
   <!-- laser Scanner laserscanner S300 optic-->
-  <joint name="${base_name}_lidar_front_right_joint" type="fixed">
+  <joint name="${base_name}_scan_front_right_joint" type="fixed">
       <parent link="${base_name}_base_link" />
-      <child link="${base_name}_lidar_front_right_link" />
+      <child link="${base_name}_scan_front_right_link" />
       <origin xyz="0.464 -0.256 0.15" rpy="0 0 -0.7854"/>
   </joint>
-  <link name="${base_name}_lidar_front_right_link"></link>
-  <joint name="${base_name}_lidar_back_left_joint" type="fixed">
+  <link name="${base_name}_scan_front_right_link"></link>
+  <joint name="${base_name}_scan_back_left_joint" type="fixed">
       <parent link="${base_name}_base_link" />
-      <child link="${base_name}_lidar_back_left_link" />
+      <child link="${base_name}_scan_back_left_link" />
       <origin xyz="-0.464 0.256 0.15" rpy="0 0 2.3562"/>
   </joint>
-  <link name="${base_name}_lidar_back_left_link"></link>
+  <link name="${base_name}_scan_back_left_link"></link>
   </xacro:macro>
 </robot>

Commit message: remove diff arm/base name, use macro avoiding copy paste

File: kmr_iiwa_gazebo/urdf/kmr_iiwa.urdf.xacro (robot description, xacro)
@@ -1,5 +1,5 @@
 <?xml version="1.0"?>
 <robot name="kmr" xmlns:xacro="http://www.ros.org/wiki/xacro">
-  <xacro:include filename="$(find kmr_iiwa_urdf)/urdf/kmp200_macro.urdf.xacro"/>
+  <xacro:include filename="$(find kmr_iiwa_urdf)/urdf/kmr_iiwa_macro.urdf.xacro"/>
   <xacro:include filename="$(find lbr_iiwa14_r820_description)/urdf/lbr_iiwa14_r820_macro.xacro" />
   <xacro:include filename="$(find lbr_ros2_control)/urdf/lbr_gazebo.xacro" />
@@ -9,6 +9,4 @@
   <xacro:arg name="root_link" default="world"/> <!-- Put world for the gazebo model, odom for nav2 -->
   <xacro:arg name="robot_name" default="kmr_iiwa" />
-  <xacro:arg name="base_name" default="kmp" />
-  <xacro:arg name="arm_name" default="iiwa" />
   <xacro:arg name="mode" default="gazebo" />
   <xacro:arg
@@ -19,12 +17,5 @@
       default="$(find lbr_ros2_control)/config/initial_joint_positions.yaml" />
   <!-- ROBOT -->
-  <xacro:kuka_kmp200 base_name="$(arg base_name)"/>
-  <xacro:lbr_iiwa14_r820
-    robot_name="$(arg robot_name)"/>
-  <joint name="$(arg base_name)_to_$(arg robot_name)_link_0" type="fixed">
-    <origin xyz="0.3633 -0.1842 0.7011" rpy="0 0 -1.5708"/>
-    <parent link="$(arg base_name)_base_link"/>
-    <child link="$(arg robot_name)_link_0"/>
-  </joint>
+  <xacro:kuka_kmr_iiwa robot_name="$(arg robot_name)"/>
   <!-- gaebo plugins -->
   <xacro:lbr_gazebo
@@ -65,11 +56,11 @@
   </ros2_control> -->
   <!-- OPTION 3. virtual joints, virtual base system -->
-  <xacro:virtual_base_system root_link="$(arg root_link)" base_link="$(arg base_name)_base_link"/>
+  <xacro:virtual_base_system root_link="$(arg root_link)" base_link="$(arg robot_name)_base_link"/>
   <!-- Sensors -->
-  <gazebo reference="$(arg base_name)_scan_front_right_link">
+  <gazebo reference="$(arg robot_name)_scan_front_right_link">
   <sensor name="scan_front_right" type="gpu_lidar">
-      <pose relative_to='$(arg base_name)_scan_front_right_link'>0 0 0 0 0 0</pose>
+      <pose relative_to='$(arg robot_name)_scan_front_right_link'>0 0 0 0 0 0</pose>
       <topic>$(arg robot_name)/scan_front_right</topic>
-      <gz_frame_id>$(arg base_name)_scan_front_right_link</gz_frame_id>
+      <gz_frame_id>$(arg robot_name)_scan_front_right_link</gz_frame_id>
       <!-- Response time 80 ms -->
       <update_rate>12.5</update_rate>
@@ -103,9 +94,9 @@
   </sensor>
   </gazebo>
-  <gazebo reference="$(arg base_name)_scan_back_left_link">
+  <gazebo reference="$(arg robot_name)_scan_back_left_link">
   <sensor name="scan_back_left" type="gpu_lidar">
-      <pose relative_to='$(arg base_name)_scan_back_left_link'>0 0 0 0 0 0</pose>
+      <pose relative_to='$(arg robot_name)_scan_back_left_link'>0 0 0 0 0 0</pose>
       <topic>$(arg robot_name)/scan_back_left</topic>
-      <gz_frame_id>$(arg base_name)_scan_back_left_link</gz_frame_id>
+      <gz_frame_id>$(arg robot_name)_scan_back_left_link</gz_frame_id>
       <!-- Response time 80 ms -->
       <update_rate>12.5</update_rate>
